File: gatorBytes_button_board.brd (EAGLE design)
At the start: 100.3 x 49.5 mm, 43 parts

Commit message: pre design review
Parts:
- removed U$30: (no value), 003:GATORBYTES6
- U$10, U$11, U$12, U$14, U$15, U$16, U$17, U$19: value GATOR_MINI -> GATOR; device TAB:GATOR_MINI -> SparkFun-Connectors:GATOR
- moved U$14 11.4 mm to (62.2, 19.1)
- moved U$17 8.89 mm to (14.0, 16.5)
- moved U$19 8.89 mm to (38.1, 16.5)
- moved U$12 8.13 mm to (86.4, 13.8)
- moved LOGO7 6.35 mm to (80.6, 47.0)
- moved LOGO8 6.35 mm to (92.5, 48.1)
- moved U$15 6.35 mm to (62.2, 35.6)
- moved U$13 5.85 mm to (64.8, 22.2)
- moved LOGO4 5.72 mm to (32.4, 45.1)
- moved LOGO3 5.71 mm to (44.3, 46.4)
- moved LOGO5 5.71 mm to (20.2, 46.4)
- moved U$10 3.81 mm to (38.1, 38.1)
- moved U$11 3.81 mm to (14.0, 38.1)
- moved LOGO1 3.18 mm to (56.5, 42.5)
- moved S1 3.18 mm to (14.0, 27.3)
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Connections:
- net N$1: now also U$19.P$1, U$19.P$2; no longer U$19.P1
- net N$2: now also U$10.P$1, U$10.P$2; no longer U$10.P1
- net N$3: now also U$17.P$1, U$17.P$2; no longer U$17.P1
- net N$4: now also U$11.P$1, U$11.P$2; no longer U$11.P1
- net N$5: now also U$16.P$1, U$16.P$2; no longer U$16.P1
- net N$6: now also U$12.P$1, U$12.P$2; no longer U$12.P1
- net N$7: now also U$15.P$1, U$15.P$2; no longer U$15.P1
- net N$9: now also U$14.P$1, U$14.P$2; no longer U$14.P1
Routing:
- net N$5: track 5.33 -> 11.8 mm
- net N$6: track 5.33 -> 10.7 mm
- net N$9: track 11.2 -> 13.9 mm
- net N$3: track 11.9 -> 14.4 mm
- net N$1: track 11.9 -> 14.4 mm
- net N$2: track 13.6 -> 15.8 mm
- net N$4: track 13.1 -> 14.4 mm
- net N$7: track 18.7 -> 17.7 mm
Other:
- board size 100.3 x 49.5 mm -> 100.3 x 54.6 mm

Commit message: post design review
Parts:
- added U$22: (no value), gator#PNG (6):GATOR#PNG
- added U$23: (no value), buzzard_labels (5):GATOR#CONTROL0
- added U$24: (no value), SparkFun-Aesthetics:SFE_LOGO_NAME_FLAME_.1
Other:
- outline, holes or cut-outs redrawn
- board text added: "v02"
- board text removed: "v01"

Commit message: post checklist changes
Parts:
- moved LOGO6 5.08 mm to (8.13, 45.1)
Routing:
- net N$7: track 17.7 -> 26.8 mm
- net N$4: track 14.4 -> 20.5 mm
- net N$2: track 15.8 -> 21.9 mm
- net N$1: track 14.4 -> 20.2 mm
- net N$3: track 14.4 -> 20.2 mm
- net N$9: track 13.9 -> 15.9 mm
- net N$6: track 10.7 -> 12.3 mm
Other:
- board text added: "v10"
- board text removed: "v02"
Changed lines of the file:
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@@
 <hole x="77.47" y="26.797" drill="0.381"/>
 <hole x="77.47" y="27.813" drill="0.381"/>
-<wire x1="1.27" y1="0" x2="0" y2="1.27" width="0.1524" layer="20" curve="-90"/>
-<wire x1="0" y1="1.27" x2="0" y2="53.34" width="0.1524" layer="20"/>
-<wire x1="0" y1="53.34" x2="1.27" y2="54.61" width="0.1524" layer="20" curve="-90"/>
-<wire x1="1.27" y1="54.61" x2="99.06" y2="54.61" width="0.1524" layer="20"/>
-<wire x1="99.06" y1="54.61" x2="100.33" y2="53.34" width="0.1524" layer="20" curve="-90"/>
-<wire x1="100.33" y1="53.34" x2="100.33" y2="1.27" width="0.1524" layer="20"/>
-<wire x1="100.33" y1="1.27" x2="99.06" y2="0" width="0.1524" layer="20" curve="-90"/>
-<wire x1="99.06" y1="0" x2="1.27" y2="0" width="0.1524" layer="20"/>
-<text x="97.79" y="0" size="1.778" layer="16" font="vector" ratio="15" rot="MR0">v02</text>
+<wire x1="1.27" y1="0" x2="0" y2="1.27" width="0.2032" layer="20" curve="-90"/>
+<wire x1="0" y1="1.27" x2="0" y2="53.34" width="0.2032" layer="20"/>
+<wire x1="0" y1="53.34" x2="1.27" y2="54.61" width="0.2032" layer="20" curve="-90"/>
+<wire x1="1.27" y1="54.61" x2="99.06" y2="54.61" width="0.2032" layer="20"/>
+<wire x1="99.06" y1="54.61" x2="100.33" y2="53.34" width="0.2032" layer="20" curve="-90"/>
+<wire x1="100.33" y1="53.34" x2="100.33" y2="1.27" width="0.2032" layer="20"/>
+<wire x1="100.33" y1="1.27" x2="99.06" y2="0" width="0.2032" layer="20" curve="-90"/>
+<wire x1="99.06" y1="0" x2="1.27" y2="0" width="0.2032" layer="20"/>
+<text x="97.79" y="0" size="1.778" layer="16" font="vector" ratio="15" rot="MR0">v10</text>
 <text x="49.53" y="-9.525" size="1.778" layer="51" font="vector" ratio="15">M. West</text>
 <text x="6.4135" y="4.7625" size="0.8128" layer="51" font="vector" ratio="15">route out</text>
@@
 <element name="LOGO4" library="SparkFun-Aesthetics" library_urn="urn:adsk.eagle:library:507" package="SFE_LOGO_FLAME_.1" package3d_urn="urn:adsk.eagle:package:37114/1" value="SFE_LOGO_FLAME.1_INCH" x="32.385" y="45.085" rot="MR0"/>
 <element name="LOGO5" library="SparkFun-Aesthetics" library_urn="urn:adsk.eagle:library:507" package="OSHW-LOGO-S" package3d_urn="urn:adsk.eagle:package:37099/1" value="OSHW-LOGOS" x="20.193" y="46.355" rot="MR0"/>
-<element name="LOGO6" library="SparkFun-Aesthetics" library_urn="urn:adsk.eagle:library:507" package="SFE_LOGO_FLAME_.1" package3d_urn="urn:adsk.eagle:package:37114/1" value="SFE_LOGO_FLAME.1_INCH" x="8.128" y="40.005" rot="MR0"/>
+<element name="LOGO6" library="SparkFun-Aesthetics" library_urn="urn:adsk.eagle:library:507" package="SFE_LOGO_FLAME_.1" package3d_urn="urn:adsk.eagle:package:37114/1" value="SFE_LOGO_FLAME.1_INCH" x="8.128" y="45.085" rot="MR0"/>
 <element name="U$33" library="SparkFun-Aesthetics" package="ORDERING_INSTRUCTIONS" value="" x="-3.81" y="-12.065"/>
 <element name="S1" library="SparkFun-Switches" package="TACTILE_SWITCH_SMD_12MM" value="MOMENTARY-SWITCH-SPST-SMD-12MM" x="13.97" y="27.305">
@@
 <wire x1="38.1" y1="22.86" x2="40.045" y2="24.805" width="0.4064" layer="1"/>
 <wire x1="40.045" y1="24.805" x2="45.075" y2="24.805" width="0.4064" layer="1"/>
-<wire x1="38.1" y1="10.414" x2="38.1" y2="16.256" width="0" layer="19" extent="1-1"/>
+<wire x1="38.1" y1="16.256" x2="38.1" y2="10.414" width="0.2032" layer="1"/>
 </signal>
 <signal name="N$2">
@@
 <wire x1="45.075" y1="29.805" x2="40.045" y2="29.805" width="0.4064" layer="1"/>
 <wire x1="40.045" y1="29.805" x2="38.1" y2="31.75" width="0.4064" layer="1"/>
-<wire x1="38.1" y1="31.75" x2="38.1" y2="38.354" width="0.4064" layer="1"/>
-<wire x1="38.1" y1="38.354" x2="38.1" y2="42.7675" width="0" layer="19" extent="1-1"/>
+<wire x1="38.1" y1="31.75" x2="38.1" y2="38.1" width="0.4064" layer="1"/>
+<wire x1="38.1" y1="44.196" x2="38.1" y2="38.1" width="0.2032" layer="1"/>
+<wire x1="38.1" y1="38.354" x2="38.1" y2="38.1" width="0.2032" layer="1"/>
 </signal>
 <signal name="N$3">
@@
 <wire x1="15.915" y1="24.805" x2="13.97" y2="22.86" width="0.4064" layer="1"/>
 <wire x1="13.97" y1="22.86" x2="13.97" y2="16.256" width="0.4064" layer="1"/>
-<wire x1="13.97" y1="10.414" x2="13.97" y2="16.256" width="0" layer="19" extent="1-1"/>
+<wire x1="13.97" y1="16.256" x2="13.97" y2="10.414" width="0.2032" layer="1"/>
 </signal>
 <signal name="N$4">
@@
 <wire x1="20.945" y1="29.805" x2="15.915" y2="29.805" width="0.4064" layer="1"/>
 <wire x1="15.915" y1="29.805" x2="13.97" y2="31.75" width="0.4064" layer="1"/>
-<wire x1="13.97" y1="31.75" x2="13.97" y2="38.354" width="0.4064" layer="1"/>
-<wire x1="13.97" y1="38.354" x2="13.97" y2="44.196" width="0" layer="19" extent="1-1"/>
+<wire x1="13.97" y1="31.75" x2="13.97" y2="38.1" width="0.4064" layer="1"/>
+<wire x1="13.97" y1="44.196" x2="13.97" y2="38.1" width="0.2032" layer="1"/>
+<wire x1="13.97" y1="38.354" x2="13.97" y2="38.1" width="0.2032" layer="1"/>
 </signal>
 <signal name="N$5">
@@
 <wire x1="86.36" y1="40.64" x2="86.36" y2="46.736" width="0.4064" layer="1"/>
 <wire x1="86.36" y1="36.195" x2="86.36" y2="40.64" width="0.4064" layer="1"/>
-<wire x1="86.36" y1="40.64" x2="86.36" y2="40.894" width="0" layer="19" extent="1-1"/>
+<wire x1="86.36" y1="40.894" x2="86.36" y2="40.64" width="0.2032" layer="1"/>
 </signal>
 <signal name="N$6">
@@
 <contactref element="U$12" pad="P$1"/>
 <contactref element="U$12" pad="P$2"/>
-<wire x1="86.36" y1="18.415" x2="86.36" y2="7.747" width="0.4064" layer="1"/>
-<wire x1="86.36" y1="18.415" x2="86.36" y2="13.589" width="0" layer="19" extent="1-1"/>
+<wire x1="86.36" y1="18.415" x2="86.36" y2="15.24" width="0.4064" layer="1"/>
+<wire x1="86.36" y1="15.24" x2="86.36" y2="7.747" width="0.4064" layer="1"/>
+<wire x1="86.36" y1="13.589" x2="86.36" y2="15.24" width="0.4064" layer="1"/>
 </signal>
 <signal name="N$7">
 <contactref element="S3" pad="2"/>
 <contactref element="U$15" pad="P$1"/>
-<wire x1="63.5" y1="38.735" x2="62.1115875" y2="38.735" width="0.4064" layer="1"/>
 <wire x1="60.96" y1="38.735" x2="61.976" y2="38.735" width="0.4064" layer="1"/>
 <contactref element="U$15" pad="P$2"/>
-<wire x1="62.1115875" y1="42.816178125" x2="62.226775" y2="42.7031375" width="0.4064" layer="1"/>
 <wire x1="62.103" y1="38.735" x2="61.976" y2="38.735" width="0.4064" layer="1"/>
-<wire x1="62.228925" y1="41.656" x2="62.226775" y2="42.7031375" width="0.4064" layer="1"/>
 <wire x1="62.1115875" y1="38.735" x2="62.103" y2="38.735" width="0.4064" layer="1"/>
 <wire x1="65.055" y1="27.305" x2="66.675" y2="27.305" width="0.4064" layer="1"/>
@@
 <wire x1="63.5" y1="31.75" x2="62.23" y2="33.02" width="0.4064" layer="1"/>
 <wire x1="62.23" y1="33.02" x2="62.23" y2="35.814" width="0.4064" layer="1"/>
-<wire x1="62.228925" y1="41.656" x2="62.23" y2="41.656" width="0" layer="19" extent="1-1"/>
-<wire x1="62.1115875" y1="38.735" x2="62.23" y2="41.656" width="0" layer="19" extent="1-1"/>
-<wire x1="62.23" y1="35.814" x2="62.1115875" y2="38.735" width="0" layer="19" extent="1-1"/>
+<wire x1="62.23" y1="41.656" x2="62.23" y2="33.02" width="0.2032" layer="1"/>
+<wire x1="62.23" y1="41.656" x2="62.23" y2="38.989" width="0.2032" layer="1"/>
+<wire x1="62.23" y1="38.989" x2="61.976" y2="38.735" width="0.2032" layer="1"/>
 </signal>
 <signal name="N$8">
@@
 <wire x1="63.5" y1="24.765" x2="62.23" y2="23.495" width="0.4064" layer="1"/>
 <contactref element="U$14" pad="P$2"/>
-<wire x1="62.23" y1="23.495" x2="62.23" y2="12.954003125" width="0.4064" layer="1"/>
-<wire x1="62.23" y1="23.495" x2="62.23" y2="18.796" width="0" layer="19" extent="1-1"/>
-<wire x1="62.23" y1="12.954" x2="62.23" y2="12.954003125" width="0" layer="19" extent="1-1"/>
+<wire x1="62.23" y1="23.495" x2="62.23" y2="17.78" width="0.4064" layer="1"/>
+<wire x1="62.23" y1="18.796" x2="62.23" y2="17.78" width="0.4064" layer="1"/>
+<wire x1="62.23" y1="18.796" x2="62.23" y2="12.954" width="0.4064" layer="1"/>
 </signal>
 </signals>

Commit message: post qc review
Parts:
- added LOGO9: REVISION, SparkFun-Aesthetics:REVISION
- moved U$23 11.5 mm to (49.5, 51.4)
Other:
- board text added: "A. England"
Changed lines of the file:
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@@
 <text x="97.79" y="0" size="1.778" layer="16" font="vector" ratio="15" rot="MR0">v10</text>
 <text x="49.53" y="-9.525" size="1.778" layer="51" font="vector" ratio="15">M. West</text>
-<text x="6.4135" y="4.7625" size="0.8128" layer="51" font="vector" ratio="15">route out</text>
+<text x="6.4135" y="4.7625" size="0.8128" layer="20" font="vector" ratio="15">route out</text>
 <text x="4.15925" y="-31.1785" size="2.54" layer="51">Solder Mask: Black Gloss</text>
 <wire x1="21.59" y1="48.895" x2="22.86" y2="47.625" width="0.2032" layer="20" curve="-90"/>
@@
 <wire x1="24.13" y1="48.895" x2="22.86" y2="50.165" width="0.2032" layer="51" curve="90"/>
 <wire x1="22.86" y1="50.165" x2="15.24" y2="50.165" width="0.2032" layer="51"/>
-<text x="16.5735" y="4.7625" size="0.8128" layer="51" font="vector" ratio="15">route out</text>
-<text x="4.7625" y="14.6685" size="0.8128" layer="51" font="vector" ratio="15" rot="R90">route out</text>
-<text x="23.8125" y="15.9385" size="0.8128" layer="51" font="vector" ratio="15" rot="R90">route out</text>
-<text x="4.7625" y="29.9085" size="0.8128" layer="51" font="vector" ratio="15" rot="R90">route out</text>
-<text x="23.8125" y="29.9085" size="0.8128" layer="51" font="vector" ratio="15" rot="R90">route out</text>
-<text x="16.5735" y="49.2125" size="0.8128" layer="51" font="vector" ratio="15">route out</text>
-<text x="11.3665" y="49.8475" size="0.8128" layer="51" font="vector" ratio="15" rot="R180">route out</text>
-<text x="30.5435" y="4.7625" size="0.8128" layer="51" font="vector" ratio="15">route out</text>
+<text x="16.5735" y="4.7625" size="0.8128" layer="20" font="vector" ratio="15">route out</text>
+<text x="4.7625" y="14.6685" size="0.8128" layer="20" font="vector" ratio="15" rot="R90">route out</text>
+<text x="23.8125" y="15.9385" size="0.8128" layer="20" font="vector" ratio="15" rot="R90">route out</text>
+<text x="4.7625" y="29.9085" size="0.8128" layer="20" font="vector" ratio="15" rot="R90">route out</text>
+<text x="23.8125" y="29.9085" size="0.8128" layer="20" font="vector" ratio="15" rot="R90">route out</text>
+<text x="16.5735" y="49.2125" size="0.8128" layer="20" font="vector" ratio="15">route out</text>
+<text x="11.3665" y="49.8475" size="0.8128" layer="20" font="vector" ratio="15" rot="R180">route out</text>
+<text x="30.5435" y="4.7625" size="0.8128" layer="20" font="vector" ratio="15">route out</text>
 <wire x1="45.72" y1="48.895" x2="46.99" y2="47.625" width="0.2032" layer="20" curve="-90"/>
 <wire x1="46.99" y1="6.985" x2="45.72" y2="5.715" width="0.2032" layer="20" curve="-90"/>
@@
 <wire x1="48.26" y1="48.895" x2="46.99" y2="50.165" width="0.2032" layer="51" curve="90"/>
 <wire x1="46.99" y1="50.165" x2="39.37" y2="50.165" width="0.2032" layer="51"/>
-<text x="40.7035" y="4.7625" size="0.8128" layer="51" font="vector" ratio="15">route out</text>
-<text x="28.8925" y="14.6685" size="0.8128" layer="51" font="vector" ratio="15" rot="R90">route out</text>
-<text x="47.9425" y="15.9385" size="0.8128" layer="51" font="vector" ratio="15" rot="R90">route out</text>
-<text x="28.8925" y="29.9085" size="0.8128" layer="51" font="vector" ratio="15" rot="R90">route out</text>
-<text x="47.9425" y="29.9085" size="0.8128" layer="51" font="vector" ratio="15" rot="R90">route out</text>
-<text x="40.7035" y="49.2125" size="0.8128" layer="51" font="vector" ratio="15">route out</text>
-<text x="35.4965" y="49.8475" size="0.8128" layer="51" font="vector" ratio="15" rot="R180">route out</text>
-<text x="54.6735" y="7.3025" size="0.8128" layer="51" font="vector" ratio="15">route out</text>
+<text x="40.7035" y="4.7625" size="0.8128" layer="20" font="vector" ratio="15">route out</text>
+<text x="28.8925" y="14.6685" size="0.8128" layer="20" font="vector" ratio="15" rot="R90">route out</text>
+<text x="47.9425" y="15.9385" size="0.8128" layer="20" font="vector" ratio="15" rot="R90">route out</text>
+<text x="28.8925" y="29.9085" size="0.8128" layer="20" font="vector" ratio="15" rot="R90">route out</text>
+<text x="47.9425" y="29.9085" size="0.8128" layer="20" font="vector" ratio="15" rot="R90">route out</text>
+<text x="40.7035" y="49.2125" size="0.8128" layer="20" font="vector" ratio="15">route out</text>
+<text x="35.4965" y="49.8475" size="0.8128" layer="20" font="vector" ratio="15" rot="R180">route out</text>
+<text x="54.6735" y="7.3025" size="0.8128" layer="20" font="vector" ratio="15">route out</text>
 <wire x1="69.85" y1="46.355" x2="71.12" y2="45.085" width="0.2032" layer="20" curve="-90"/>
 <wire x1="71.12" y1="9.525" x2="69.85" y2="8.255" width="0.2032" layer="20" curve="-90"/>
@@
 <wire x1="72.39" y1="46.355" x2="71.12" y2="47.625" width="0.2032" layer="51" curve="90"/>
 <wire x1="71.12" y1="47.625" x2="63.5" y2="47.625" width="0.2032" layer="51"/>
-<text x="64.8335" y="7.3025" size="0.8128" layer="51" font="vector" ratio="15">route out</text>
-<text x="53.0225" y="17.2085" size="0.8128" layer="51" font="vector" ratio="15" rot="R90">route out</text>
-<text x="72.0725" y="18.4785" size="0.8128" layer="51" font="vector" ratio="15" rot="R90">route out</text>
-<text x="53.0225" y="29.9085" size="0.8128" layer="51" font="vector" ratio="15" rot="R90">route out</text>
-<text x="72.0725" y="29.9085" size="0.8128" layer="51" font="vector" ratio="15" rot="R90">route out</text>
-<text x="64.8335" y="46.6725" size="0.8128" layer="51" font="vector" ratio="15">route out</text>
-<text x="59.6265" y="47.3075" size="0.8128" layer="51" font="vector" ratio="15" rot="R180">route out</text>
-<text x="78.8035" y="2.2225" size="0.8128" layer="51" font="vector" ratio="15">route out</text>
+<text x="64.8335" y="7.3025" size="0.8128" layer="20" font="vector" ratio="15">route out</text>
+<text x="53.0225" y="17.2085" size="0.8128" layer="20" font="vector" ratio="15" rot="R90">route out</text>
+<text x="72.0725" y="18.4785" size="0.8128" layer="20" font="vector" ratio="15" rot="R90">route out</text>
+<text x="53.0225" y="29.9085" size="0.8128" layer="20" font="vector" ratio="15" rot="R90">route out</text>
+<text x="72.0725" y="29.9085" size="0.8128" layer="20" font="vector" ratio="15" rot="R90">route out</text>
+<text x="64.8335" y="46.6725" size="0.8128" layer="20" font="vector" ratio="15">route out</text>
+<text x="59.6265" y="47.3075" size="0.8128" layer="20" font="vector" ratio="15" rot="R180">route out</text>
+<text x="78.8035" y="2.2225" size="0.8128" layer="20" font="vector" ratio="15">route out</text>
 <wire x1="93.98" y1="51.435" x2="95.25" y2="50.165" width="0.2032" layer="20" curve="-90"/>
 <wire x1="95.25" y1="4.445" x2="93.98" y2="3.175" width="0.2032" layer="20" curve="-90"/>
@@
 <wire x1="96.52" y1="51.435" x2="95.25" y2="52.705" width="0.2032" layer="51" curve="90"/>
 <wire x1="95.25" y1="52.705" x2="87.63" y2="52.705" width="0.2032" layer="51"/>
-<text x="88.9635" y="2.2225" size="0.8128" layer="51" font="vector" ratio="15">route out</text>
-<text x="77.1525" y="18.4785" size="0.8128" layer="51" font="vector" ratio="15" rot="R90">route out</text>
-<text x="96.2025" y="19.7485" size="0.8128" layer="51" font="vector" ratio="15" rot="R90">route out</text>
-<text x="77.1525" y="29.9085" size="0.8128" layer="51" font="vector" ratio="15" rot="R90">route out</text>
-<text x="96.2025" y="29.9085" size="0.8128" layer="51" font="vector" ratio="15" rot="R90">route out</text>
-<text x="88.9635" y="51.7525" size="0.8128" layer="51" font="vector" ratio="15">route out</text>
-<text x="83.7565" y="52.3875" size="0.8128" layer="51" font="vector" ratio="15" rot="R180">route out</text>
+<text x="88.9635" y="2.2225" size="0.8128" layer="20" font="vector" ratio="15">route out</text>
+<text x="77.1525" y="18.4785" size="0.8128" layer="20" font="vector" ratio="15" rot="R90">route out</text>
+<text x="96.2025" y="19.7485" size="0.8128" layer="20" font="vector" ratio="15" rot="R90">route out</text>
+<text x="77.1525" y="29.9085" size="0.8128" layer="20" font="vector" ratio="15" rot="R90">route out</text>
+<text x="96.2025" y="29.9085" size="0.8128" layer="20" font="vector" ratio="15" rot="R90">route out</text>
+<text x="88.9635" y="51.7525" size="0.8128" layer="20" font="vector" ratio="15">route out</text>
+<text x="83.7565" y="52.3875" size="0.8128" layer="20" font="vector" ratio="15" rot="R180">route out</text>
 <hole x="53.34" y="26.797" drill="0.381"/>
 <hole x="53.34" y="27.813" drill="0.381"/>
@@
 <hole x="96.52" y="27.813" drill="0.381"/>
 <hole x="96.52" y="26.797" drill="0.381"/>
+<text x="48.514" y="-11.684" size="1.778" layer="51" font="vector" ratio="15">A. England</text>
 </plain>
 <attributes>
@@
 <element name="U$21" library="buzzard_labels (3)" package="SWITCH5" value="" x="81.28" y="26.035" rot="MR90"/>
 <element name="U$22" library="gator#PNG (6)" package="GATOR#PNG" value="" x="68.5165" y="3.6195"/>
-<element name="U$23" library="buzzard_labels (5)" package="GATOR#CONTROL0" value="" x="38.1" y="52.705"/>
+<element name="U$23" library="buzzard_labels (5)" package="GATOR#CONTROL0" value="" x="49.53" y="51.435"/>
 <element name="U$24" library="SparkFun-Aesthetics" package="SFE_LOGO_NAME_FLAME_.1" value="" x="51.689" y="1.27"/>
+<element name="LOGO9" library="SparkFun-Aesthetics" package="REVISION" value="REVISION" x="33.782" y="-11.557"/>
 </elements>
 <signals>
